File: plant-sensor.kicad_pcb (KiCad board)
At the start: 2 copper layers, 43 parts, among them J1 Conn_01x02_Male, J2 Conn_01x05_Male, Q2 MMBT3904, Q3 MMBT3904, SW1 SW_Push, SW2 SW_Push, U2 STM32L031F4Px

Commit message: version sent to jlc
Parts:
- removed C10, C11, C12, C13, C14, C15, C16, C2, C3, C4, C5, C7, C9: 1uF, Capacitor_SMD:C_0603_1608Metric_Pad1.05x0.95mm_HandSolder
- removed C17, C20, C21: 0.1uF, Capacitor_SMD:C_0603_1608Metric_Pad1.05x0.95mm_HandSolder
- removed C6, C8: 2.2uF, Capacitor_SMD:C_0603_1608Metric_Pad1.05x0.95mm_HandSolder
- removed D1: MBR0530, Diode_SMD:D_SOD-123
- removed FPC1: Conn_01x30_Male, Connector_FFC-FPC:TE_2-1734839-9_1x29-1MP_P0.5mm_Horizontal
- removed R3, R4: 10k, Resistor_SMD:R_0603_1608Metric_Pad1.05x0.95mm_HandSolder
- removed SW1, SW2: SW_Push, Button_Switch_SMD:SW_SPST_B3S-1000
- added J3: Conn_01x03_Male, Connector_PinHeader_2.54mm:PinHeader_1x03_P2.54mm_Vertical, B.Cu at (50.0, 80.0)
- added J4: Conn_01x03_Male, Connector_PinHeader_2.54mm:PinHeader_1x03_P2.54mm_Vertical, B.Cu at (73.4, 80.0)
- added J5: Conn_01x01_Male, Connector_PinHeader_2.54mm:PinHeader_1x01_P2.54mm_Vertical, B.Cu at (50.0, 111.0)
- added J6: Conn_01x01_Male, Connector_PinHeader_2.54mm:PinHeader_1x01_P2.54mm_Vertical, B.Cu at (73.4, 111.0)
- C1: value 4.7uF -> 100n
- C18: footprint Capacitor_SMD:C_0603_1608Metric_Pad1.05x0.95mm_HandSolder -> Capacitor_SMD:C_1206_3216Metric_Pad1.42x1.75mm_HandSolder
- C25, C26, C27, C28, D3, Q2, Q3, R10, R11, R12, R13, R14, U2: moved to B.Cu
- R9: value R -> 10k; moved to B.Cu
- moved J2 74.2 mm to (56.0, 78.3), turned to 90 degrees
- moved J1 60.9 mm to (50.0, 103.5), turned to 0 degrees
- moved C1 56.4 mm to (70.5, 76.8)
- moved R14 55.3 mm to (53.0, 104.9)
- moved R12 53.5 mm to (55.0, 100.3)
- moved R9 52.7 mm to (56.1, 87.6), turned to 180 degrees
- moved Q3 52.4 mm to (56.6, 105.6), turned to 180 degrees
- moved R11 51.8 mm to (57.5, 100.3)
- moved C25 51.3 mm to (58.4, 97.7), turned to 180 degrees
- moved C26 50.6 mm to (60.0, 100.3)
- moved U2 50.6 mm to (60.0, 92.6)
- moved Q2 50.1 mm to (61.6, 105.6), turned to 180 degrees
- moved R10 49.8 mm to (62.6, 100.3)
- moved C28 49.8 mm to (67.3, 88.8), turned to 0 degrees
- moved C27 49.8 mm to (67.3, 101.5), turned to 180 degrees
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Connections:
- C1 pad 1: VCC -> /RESET
- C27 pad 1: Net-(C27-Pad1) -> /Csen+
- D3 pad 2: Net-(C27-Pad1) -> /Csen+
- R10 pad 1: Net-(C27-Pad1) -> /Csen+
- U2 pad 14: /MODE_BUTTON -> Net-(U2-Pad14)
Routing:
- net VCC: track 0.00 -> 132.9 mm, vias 0 -> 1
- net /Csen+: track 0.00 -> 112.4 mm
- net /SWDIO: track 0.00 -> 27.4 mm
- net /CS: track 0.00 -> 27.3 mm, vias 0 -> 1
- net /SWCLK: track 0.00 -> 25.1 mm
- net /FAST_DISCH_EN: track 0.00 -> 24.8 mm, vias 0 -> 2
- net GND: track 0.00 -> 21.4 mm, vias 0 -> 9
- net /CLK: track 0.00 -> 20.9 mm, vias 0 -> 1
- net /RX: track 0.00 -> 20.1 mm
- net /SENS_OUT: track 0.00 -> 18.5 mm
- net /RESET: track 0.00 -> 18.5 mm
- net /TX: track 0.00 -> 17.9 mm
- net /MOSI: track 0.00 -> 17.7 mm, vias 0 -> 1
- net /DC: track 0.00 -> 16.2 mm
- net /RST: track 0.00 -> 14.5 mm
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- added copper zone on B.Cu, net GND
- added copper zone on F.Cu, net GND
Other:
- board outline added: 27.4 x 116.2 mm
- board text added: "+"
- board text added: "-"
- board text added: "BUSY"
- board text added: "CETTE PARTIE DANS LA TERRE"
- board text added: "CLK"
- board text added: "CS"
- board text added: "DC"
- board text added: "DIO"
- board text added: "Fait avec amour par le Chouchou"
- board text added: "GND"
- board text added: "La capteur d’humidité pour la Chacha"
- board text added: "MOSI"
- board text added: "RST"
- board text added: "VCC"

Commit message: changes
Other:
- board text added: "JLCJLCJLCJLC"
Changed lines of the file:
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@@
   (general
     (thickness 1.6)
-    (drawings 32)
+    (drawings 33)
     (tracks 171)
     (zones 0)
@@
       (outputformat 1)
       (mirror false)
-      (drillshape 1)
+      (drillshape 0)
       (scaleselection 1)
       (outputdirectory ""))
@@
       (effects (font (size 0.8 0.8) (thickness 0.12)))
     )
-    (pad 2 smd roundrect (at 1.4875 0) (size 1.425 1.75) (layers F.Cu F.Paste F.Mask) (roundrect_rratio 0.175439)
+    (pad 2 smd roundrect (at 1.4875 0) (size 1.425 1.75) (layers F.Cu F.Paste F.Mask) (roundrect_rratio 0.1754385964912281)
       (net 2 VCC))
-    (pad 1 smd roundrect (at -1.4875 0) (size 1.425 1.75) (layers F.Cu F.Paste F.Mask) (roundrect_rratio 0.175439)
+    (pad 1 smd roundrect (at -1.4875 0) (size 1.425 1.75) (layers F.Cu F.Paste F.Mask) (roundrect_rratio 0.1754385964912281)
       (net 1 GND))
     (model ${KISYS3DMOD}/Capacitor_SMD.3dshapes/C_1206_3216Metric.wrl
@@
     )
   )
+  (gr_text JLCJLCJLCJLC (at 69 104) (layer B.SilkS)
+    (effects (font (size 1 1) (thickness 0.15)) (justify mirror))
+  )
   (gr_text "Fait avec amour par le Chouchou" (at 68 153 90) (layer F.SilkS)
