File: plant-sensor.sch (KiCad schematic (older format))
At the start: 43 parts, among them J1 Conn_01x02_Male, J2 Conn_01x05_Male, Q2 MMBT3904, Q3 MMBT3904, SW1 SW_Push, SW2 SW_Push, U2 STM32L031F4Px

Commit message: version sent to jlc
Parts:
- removed C10, C11, C12, C13, C14, C15, C16, C2, C3, C4, C5, C7, C9: 1uF, Capacitor_SMD:C_0603_1608Metric_Pad1.05x0.95mm_HandSolder, symbol Device:C
- removed C17, C20, C21: 0.1uF, Capacitor_SMD:C_0603_1608Metric_Pad1.05x0.95mm_HandSolder, symbol Device:C
- removed C6, C8: 2.2uF, Capacitor_SMD:C_0603_1608Metric_Pad1.05x0.95mm_HandSolder, symbol Device:C
- removed D1: MBR0530, Diode_SMD:D_SOD-123, symbol Diode:MBR0530
- removed FPC1: Conn_01x30_Male, Connector_FFC-FPC:TE_2-1734839-9_1x29-1MP_P0.5mm_Horizontal, symbol Connector:Conn_01x30_Male
- removed R3, R4: 10k, Resistor_SMD:R_0603_1608Metric_Pad1.05x0.95mm_HandSolder, symbol Device:R
- removed SW1, SW2: SW_Push, Button_Switch_SMD:SW_SPST_B3S-1000, symbol Switch:SW_Push
- added J3, J4: Conn_01x03_Male, Connector_PinHeader_2.54mm:PinHeader_1x03_P2.54mm_Vertical, symbol Connector:Conn_01x03_Male
- added J5, J6: Conn_01x01_Male, Connector_PinHeader_2.54mm:PinHeader_1x01_P2.54mm_Vertical, symbol Connector:Conn_01x01_Male
- C1: value 4.7uF -> 100n
- C18: footprint Capacitor_SMD:C_0603_1608Metric_Pad1.05x0.95mm_HandSolder -> Capacitor_SMD:C_1206_3216Metric_Pad1.42x1.75mm_HandSolder
- R9: value R -> 10k
Connections:
- net BUSY: now also J4.3 (Pin_3)
- net CLK: now also J3.2 (Pin_2)
- net CS: now also J3.1 (Pin_1)
- net DC: now also J4.1 (Pin_1)
- net GND: now also J6.1 (Pin_1)
- net MOSI: now also J3.3 (Pin_3)
- net RESET: now also C1.1
- net RST: now also J4.2 (Pin_2)
- net VCC: now also J5.1 (Pin_1); no longer C1.1
- net MODE_BUTTON: no longer names the net of U2.14 (PB1)

Commit message: changes
Connections:
- net Csen+: now also C27.1, D3.2 (A), R10.1
Changed lines of the file:
@@
 	1000 1200 1800 1200
 NoConn ~ 1800 2300
+Text Label 5150 1200 0    50   ~ 0
+Csen+
 $EndSCHEMATC
